File: Shield.kicad_pcb (KiCad board)
At the start: 4 copper layers, 162 x 99.6 mm, 96 parts, among them J1 SAMTEC-FTS-130-01-X-DV, J11 USB_C_Receptacle_PowerOnly_6P, J12 SIM_Card_Shielded, J13 Conn_02x03_Odd_Even, J14 USB3_A, J15 USB3_A, J16 AUDIO-SMD_PJ-342C-1, J2 SAMTEC-FTS-130-01-X-DV, J3 5051102291, J4 5051102291, J5 77313-118-40LF, J6 Bus_PCI_Express_Mini, J7 USB_C_Receptacle, J8 Bus_PCI_Express_Mini, J9 USB3_A, Q1 2N3904, Q2 MMBT3904, Q3 MMBT3904, U1 TCA9406DCUR, U10 AP62300Z6-7, U2 USB5744_2G, U3 AMS1117-3.3, U4 AMS1117-3.3, U5 AMS1117-1.8, U6 LM1117S-1.2, U7 TPS2051BDBVR, U8 TPS2051BDBVR, U9 TPS2051BDBVR, Y1 Crystal

Commit message: Updated
Parts:
- removed C32: 100 n, Capacitor_SMD:C_0805_2012Metric
- removed J16: AUDIO-SMD_PJ-342C-1, AUDIO-SMD_PJ-342C-1_PJ-3543-X_C319101:AUDIO-SMD_PJ-342C-1_PJ-3543-X_C319101
- removed R17: 2.2 K, Resistor_SMD:R_0805_2012Metric
- moved R20 211.4 mm to (34.9, 122.1), turned to 180 degrees
- moved R21 206.8 mm to (39.2, 122.0), turned to 180 degrees
- moved C36 206.5 mm to (34.9, 119.5), turned to 180 degrees
- moved C33 203.0 mm to (39.2, 119.5), turned to 180 degrees
- moved Q3 124.8 mm to (43.9, 121.9)
- moved LED2 123.2 mm to (36.9, 128.2), turned to 180 degrees
- moved R19 84.5 mm to (161.1, 105.1)
- moved R18 84.3 mm to (162.1, 109.5)
- moved C35 83.1 mm to (158.2, 109.5)
- moved C34 79.9 mm to (161.1, 102.5), turned to 180 degrees
- moved LED1 68.1 mm to (160.1, 114.4), turned to 180 degrees
- moved Q2 63.9 mm to (165.6, 106.0)
Connections:
- C35 pad 2: Net-(LED1-VDD) -> /5V-VBUS
- J2 pad 29: /MIC2_INP -> unconnected-(J2-Pad29)
- J2 pad 31: /HPH_REF -> unconnected-(J2-Pad31)
- J2 pad 33: /MIC2_BIAS -> unconnected-(J2-Pad33)
- J2 pad 36: /HPH_L -> unconnected-(J2-Pad36)
- J2 pad 38: /HPH_R -> unconnected-(J2-Pad38)
- J2 pad 40: /HPH_REF -> unconnected-(J2-Pad40)
- J5 pad 30: /SOC_GPIO_100 -> unconnected-(J5-Pad30)
- J5 pad 32: /SOC_GPIO_101 -> unconnected-(J5-Pad32)
- LED1 pad 1-VDD: Net-(LED1-VDD) -> /5V-VBUS
- R18 pad 1: Net-(LED1-VDD) -> /5V-VBUS
Routing:
- net /SOC_GPIO_18_PWM_LED: track 0.00 -> 99.3 mm, vias 0 -> 4
- net /MCU_PE8_LED: track 0.00 -> 86.6 mm, vias 0 -> 2
- net /5V-VBUS: track 283.0 -> 321.5 mm
- net (no net): track 26.6 -> 0.00 mm, vias 1 -> 0
- net /3V3-VBUS-2: track 59.6 -> 76.0 mm
- net Net-(LED2-DI): track 0.00 -> 14.3 mm
- net Net-(LED1-DI): track 0.00 -> 10.1 mm
- net /1V8: track 21.4 -> 29.9 mm
- net Net-(Q3-B): track 0.00 -> 3.30 mm
- net Net-(Q2-B): track 0.00 -> 2.64 mm
- added copper zone on In1.Cu, net GND
- added copper zone on In2.Cu, net GND
