File: Shield.kicad_sch (KiCad schematic)
At the start: 96 parts, among them J1 SAMTEC-FTS-130-01-X-DV, J11 USB_C_Receptacle_PowerOnly_6P, J12 SIM_Card_Shielded, J13 Conn_02x03_Odd_Even, J14 USB3_A, J15 USB3_A, J16 AUDIO-SMD_PJ-342C-1, J2 SAMTEC-FTS-130-01-X-DV, J3 5051102291, J4 5051102291, J5 77313-118-40LF, J6 Bus_PCI_Express_Mini, J7 USB_C_Receptacle, J8 Bus_PCI_Express_Mini, J9 USB3_A, Q1 2N3904, Q2 MMBT3904, Q3 MMBT3904, U1 TCA9406DCUR, U10 AP62300Z6-7, U2 USB5744_2G, U3 AMS1117-3.3, U4 AMS1117-3.3, U5 AMS1117-1.8, U6 LM1117S-1.2, U7 TPS2051BDBVR, U8 TPS2051BDBVR, U9 TPS2051BDBVR, Y1 Crystal

Commit message: Updated
Parts:
- removed C32: 100 n, Capacitor_SMD:C_0805_2012Metric, symbol Device:C
- removed J16: AUDIO-SMD_PJ-342C-1, AUDIO-SMD_PJ-342C-1_PJ-3543-X_C319101:AUDIO-SMD_PJ-342C-1_PJ-3543-X_C319101, symbol AUDIO_C319101:AUDIO-SMD_PJ-342C-1
- removed R17: 2.2 K, Resistor_SMD:R_0805_2012Metric, symbol Device:R_US
Connections:
- net 5V-VBUS: now also C35.2, LED1.1-VDD (VDD), R18.1
- net HPH_L: no longer names the net of J2.36
- net HPH_R: no longer names the net of J2.38
- net HPH_REF: no longer names the net of J2.31
- net HPH_REF: no longer J2.40
- net MIC2_BIAS: no longer names the net of J2.33
- net MIC2_INP: no longer names the net of J2.29
- net SOC_GPIO_100: no longer names the net of J5.30
- net SOC_GPIO_101: no longer names the net of J5.32
- no-connect marks 98 -> 102
Other:
- moved on the sheet: C33, C36, LED2, Q3, R20, R21

Commit message: PCB updated: Zero Errors
Connections:
- net UART_TXD: now reaches J8.17 (UIM_C8)
- net UART_RXD: now reaches J8.19 (UIM_C4)
- net MCU_OPAMP1_VINM / PA1: no longer names the net of J5.24
- net MCU_OPAMP1_VINM / PA1: no longer J2.24
- net MCU_OPAMP1_VINP / PA0: no longer names the net of J5.22
- net MCU_OPAMP1_VINP / PA0: no longer J2.22
- net VIN: no longer names the net of J1.59
- net VIN: no longer J5.38
- new net MCU_PA0 UART4_TX AF8: J2.22
- new net MCU_PA1 UART4_RX AF8: J2.24
- no-connect marks 102 -> 107
Changed lines of the file:
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@@
 	)
 	(no_connect
+		(at 87.63 116.84)
+	)
+	(no_connect
 		(at 505.46 77.47)
 	)
@@
 	)
 	(no_connect
-		(at 554.99 317.5)
-	)
-	(no_connect
 		(at 519.43 309.88)
 	)
@@
 	)
 	(no_connect
+		(at 529.59 175.26)
+	)
+	(no_connect
 		(at 120.65 215.9)
 	)
@@
 	)
 	(no_connect
+		(at 529.59 193.04)
+	)
+	(no_connect
 		(at 419.1 198.12)
 	)
@@
 	)
 	(no_connect
+		(at 529.59 160.02)
+	)
+	(no_connect
 		(at 541.02 102.87)
 	)
@@
 	)
 	(no_connect
-		(at 528.32 46.99)
+		(at 529.59 172.72)
 	)
 	(no_connect
-		(at 554.99 271.78)
+		(at 528.32 46.99)
 	)
 	(no_connect
-		(at 554.99 314.96)
+		(at 554.99 271.78)
 	)
 	(no_connect
@@
 	)
 	(no_connect
+		(at 529.59 182.88)
+	)
+	(no_connect
 		(at 542.29 259.08)
 	)
@@
 	)
 	(no_connect
+		(at 529.59 185.42)
+	)
+	(no_connect
 		(at 419.1 200.66)
 	)
@@
 	(wire
 		(pts
-			(xy 87.63 116.84) (xy 104.14 116.84)
-		)
-		(stroke
-			(width 0)
-			(type default)
-		)
-	)
-	(wire
-		(pts
 			(xy 316.23 257.81) (xy 316.23 255.27)
 		)
@@
 	(wire
 		(pts
-			(xy 529.59 175.26) (xy 560.07 175.26)
-		)
-		(stroke
-			(width 0)
-			(type default)
-		)
-	)
-	(wire
-		(pts
 			(xy 330.2 77.47) (xy 330.2 69.85)
 		)
@@
 	(wire
 		(pts
-			(xy 529.59 185.42) (xy 560.07 185.42)
-		)
-		(stroke
-			(width 0)
-			(type default)
-		)
-	)
-	(wire
-		(pts
 			(xy 106.68 223.52) (xy 120.65 223.52)
 		)
@@
 	(wire
 		(pts
-			(xy 529.59 182.88) (xy 560.07 182.88)
-		)
-		(stroke
-			(width 0)
-			(type default)
-		)
-	)
-	(wire
-		(pts
 			(xy 173.99 90.17) (xy 177.8 90.17)
 		)
@@
 	(wire
 		(pts
-			(xy 529.59 193.04) (xy 560.07 193.04)
-		)
-		(stroke
-			(width 0)
-			(type default)
-		)
-	)
-	(wire
-		(pts
 			(xy 313.69 378.46) (xy 313.69 387.35)
 		)
@@
 	(wire
 		(pts
+			(xy 554.99 317.5) (xy 568.96 317.5)
+		)
+		(stroke
+			(width 0)
+			(type default)
+		)
+	)
+	(wire
+		(pts
 			(xy 419.1 180.34) (xy 453.39 180.34)
 		)
@@
 	(wire
 		(pts
-			(xy 529.59 172.72) (xy 560.07 172.72)
-		)
-		(stroke
-			(width 0)
-			(type default)
-		)
-	)
-	(wire
-		(pts
 			(xy 177.8 97.79) (xy 160.02 97.79)
 		)
@@
 	(wire
 		(pts
-			(xy 529.59 160.02) (xy 560.07 160.02)
-		)
-		(stroke
-			(width 0)
-			(type default)
-		)
-	)
-	(wire
-		(pts
 			(xy 39.37 91.44) (xy 57.15 91.44)
 		)
@@
 	(wire
 		(pts
+			(xy 554.99 314.96) (xy 568.96 314.96)
+		)
+		(stroke
+			(width 0)
+			(type default)
+		)
+	)
+	(wire
+		(pts
 			(xy 57.15 104.14) (xy 52.07 104.14)
 		)
@@
 		)
 	)
-	(label "MCU_OPAMP1_VINM / PA1"
+	(label "MCU_PA1 UART4_RX AF8"
 		(at 453.39 180.34 180)
 		(effects
@@
 		)
 	)
+	(label "UART_TXD"
+		(at 568.96 317.5 180)
+		(effects
+			(font
+				(size 1.27 1.27)
+			)
+			(justify right bottom)
+		)
+	)
 	(label "MCU_PSSI_PDCK {slash} PD9"
 		(at 471.17 167.64 0)
@@
 		)
 	)
-	(label "MCU_OPAMP1_VINP / PA0"
+	(label "MCU_PA0 UART4_TX AF8"
 		(at 453.39 177.8 180)
 		(effects
@@
 		)
 	)
+	(label "UART_RXD"
+		(at 568.96 314.96 180)
+		(effects
+			(font
+				(size 1.27 1.27)
+			)
+			(justify right bottom)
+		)
+	)
 	(label "5V-VBUS"
 		(at 339.09 261.62 0)
@@
 		)
 	)
-	(label "MCU_OPAMP1_VINP / PA0"
-		(at 560.07 172.72 180)
-		(effects
-			(font
-				(size 1.27 1.27)
-			)
-			(justify right bottom)
-		)
-	)
 	(label "LR_MOSI"
 		(at 554.99 82.55 180)
@@
 		)
 	)
-	(label "VIN"
-		(at 560.07 193.04 180)
-		(effects
-			(font
-				(size 1.27 1.27)
-			)
-			(justify right bottom)
-		)
-	)
 	(label "UP_RX+"
 		(at 209.55 208.28 180)
@@
 		)
 	)
-	(label "VIN"
-		(at 104.14 116.84 180)
-		(effects
-			(font
-				(size 1.27 1.27)
-			)
-			(justify right bottom)
-		)
-	)
 	(label "MCU_I2C4_SDA / PF15"
 		(at 453.39 172.72 180)
@@
 		)
 	)
-	(label "MCU_OPAMP1_VINM / PA1"
-		(at 560.07 175.26 180)
-		(effects
-			(font
-				(size 1.27 1.27)
-			)
-			(justify right bottom)
-		)
-	)

Commit message: Added UART for LTE<->MCU
Parts:
- added U11: TXB0102DCUR, TXB0102DCUR:DCU0008A_N, symbol TXB0102DCUR:TXB0102DCUR
- J11: footprint U262-061N-4BVC10:U262-061N-4BVC10_XKB -> Type C 6 pin_ul_U262-061N-4BVC10:U262-061N-4BVC10_XKB
- U7, U8, U9: symbol 2026-06-29_17-55-01:TPS2051BDBVR -> TPS2051BDBVR:TPS2051BDBVR
Connections:
- net 1V8: now also U11.3 (VCCA)
- net GND: now also LED1.3-GND (GND), U5.1 (GND), U11.2 (GND), U11.6 (OE)
- net MCU_PA0 UART4_TX AF8: now also U11.8 (B1)
- net MCU_PA1 UART4_RX AF8: now also U11.1 (B2)
- net VDD33: now also U11.7 (VCCB)
- net SOC_GPIO_28_PWM: no longer names the net of J2.51
- net UART_RXD renamed LTE_UART_RXD
- net LTE_UART_RXD: now also U11.5 (A1)
- net UART_TXD renamed LTE_UART_TXD
- net LTE_UART_TXD: now also U11.4 (A2)
- no-connect marks 107 -> 109
Other:
- note added: "UART CONNECTION FOR LTE WITH MCU"
